File: Current Files/PCBs/TM13/TM13.kicad_pcb (KiCad board)
At the start: 2 copper layers, 76 x 76 mm, 49 parts, among them IC1 PCA9306DCUR, IC2 AZ1117, IC3 XL2596, J2 Conn_01x03_Male, J3 Conn_01x03_Male, J4 Barrel_Jack_Switch, Q1 BSS138, Q2 BSS138, Q3 BC847, Q4 BSS841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

Commit message: no auto reconnect, trim webserver input
Parts:
- removed the D4 at (77.7, 62.7)
- removed the R13 at (77.7, 58.4)
- added D1: Status, LED_SMD:LED_0805_2012Metric, F.Cu at (73.1, 67.7)
- added D2: Power, LED_SMD:LED_0805_2012Metric, F.Cu at (79.7, 67.8)
- added Q3: BC847, Package_TO_SOT_SMD:SOT-23, F.Cu at (73.0, 60.1)
- added R11: 150, Resistor_SMD:R_0603_1608Metric, F.Cu at (73.1, 64.4)
- added R12: 1K, Resistor_SMD:R_0603_1608Metric, F.Cu at (78.6, 58.4)
- renumbered D2 to D3, D3 to D4, Q3 to Q4, Q4 to Q5, R11 to R13, R12 to R14
Connections:
- U1 pad 5: unconnected-(U1-Pad5) -> GPIO14
Routing:
- net GPIO14: track 0.00 -> 29.9 mm, vias 0 -> 2
- net Net-(D2-Pad2): track 0.00 -> 8.64 mm
- net Net-(Q3-Pad2): track 0.00 -> 3.37 mm
- net Net-(D1-Pad2): track 0.00 -> 3.35 mm
- net Net-(D4-Pad2): track 2.54 -> 0.00 mm
- net +5V: track 150.6 -> 152.2 mm
- net GND: track 68.0 -> 69.6 mm, vias 23 -> 24

Commit message: update pcb
Parts:
- removed D1: Status, LED_SMD:LED_0805_2012Metric
- removed the D2 at (79.7, 67.8)
- removed J1: ~, MyFootprints:MOLEX_105133-0011
- removed the Q3 at (73.0, 60.1)
- removed the R11 at (73.1, 64.4)
- removed the R12 at (78.6, 58.4)
- added D4: LED, LED_SMD:LED_0805_2012Metric, F.Cu at (77.7, 62.7)
- added J5: 105133-0011, MyFootprints:MOLEX_105133-0011, F.Cu at (67.6, 78.3)
- added R13: 1K, Resistor_SMD:R_0603_1608Metric, F.Cu at (77.7, 58.4)
- IC2: footprint Package_TO_SOT_SMD:SOT-223 -> MyFootprints:SOT230P700X180-4N
- U4: footprint DS9503P:TSO6C -> MyFootprints:TSO6C
- renumbered D3 to D2, D4 to D3, Q4 to Q3, Q5 to Q4, R13 to R11, R14 to R12
Connections:
- U1 pad 5: GPIO14 -> unconnected-(U1-GPIO14-Pad5)
Routing:
- net GPIO14: track 29.9 -> 0.00 mm, vias 2 -> 0
- net Net-(D2-Pad2): track 8.64 -> 0.00 mm
- net Net-(Q3-Pad2): track 3.37 -> 0.00 mm
- net Net-(D1-Pad2): track 3.35 -> 0.00 mm
- net Net-(D4-A): track 0.00 -> 2.54 mm
- net GND: track 69.6 -> 68.0 mm, vias 24 -> 23
- net +5V: track 152.2 -> 150.7 mm
