File: Current Files/PCBs/TM13/TM13.kicad_sch (KiCad schematic)
At the start: 45 parts, among them IC1 PCA9306DCUR, IC2 AZ1117, IC3 XL2596, J2 Conn_01x03_Male, J3 Conn_01x03_Male, J4 Barrel_Jack_Switch, Q1 BSS138, Q2 BSS138, Q3 BC847, Q4 BSS841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

Commit message: no auto reconnect, trim webserver input
Parts:
- removed D4: LED, LED_SMD:LED_0805_2012Metric, symbol Device:LED
- removed R13: 1K, Resistor_SMD:R_0603_1608Metric, symbol Device:R
- added D1: Status, LED_SMD:LED_0805_2012Metric, symbol Device:LED
- added D2: Power, LED_SMD:LED_0805_2012Metric, symbol Device:LED
- added Q3: BC847, Package_TO_SOT_SMD:SOT-23, symbol Transistor_BJT:BC847
- added R11: 150, Resistor_SMD:R_0603_1608Metric, symbol Device:R
- added R12: 1K, Resistor_SMD:R_0603_1608Metric, symbol Device:R
- renumbered D2 to D3, D3 to D4, Q3 to Q4, Q4 to Q5, R11 to R13, R12 to R14
Connections:
- net +5V: now also Q3.3 (C), R12.1
- net GND: now also D1.1 (K), D2.1 (K)
- net GPIO14: now reaches U1.5 (GPIO14)
- net GPIO14: now also Q3.1 (B)
- new net: D2.2 (A), R12.2
- new net: D1.2 (A), R11.1
- new net: Q3.2 (E), R11.2
- no-connect marks 13 -> 12

Commit message: update pcb
Parts:
- removed D1: Status, LED_SMD:LED_0805_2012Metric, symbol Device:LED
- removed D2: Power, LED_SMD:LED_0805_2012Metric, symbol Device:LED
- removed J1: ~, MyFootprints:MOLEX_105133-0011, symbol MyLib:105133-0011-105133-0011
- removed Q3: BC847, Package_TO_SOT_SMD:SOT-23, symbol Transistor_BJT:BC847
- removed R11: 150, Resistor_SMD:R_0603_1608Metric, symbol Device:R
- removed R12: 1K, Resistor_SMD:R_0603_1608Metric, symbol Device:R
- added D4: LED, LED_SMD:LED_0805_2012Metric, symbol Device:LED
- added J5: 105133-0011, MyFootprints:MOLEX_105133-0011, symbol MyLib:105133-0011
- added R13: 1K, Resistor_SMD:R_0603_1608Metric, symbol Device:R
- IC2: footprint Package_TO_SOT_SMD:SOT-223 -> SOT230P700X180-4N; symbol MyLib:AZ1117 -> MyLib:AZ1117CH-3.3TRG1; Height (none) -> 1.8; Manufacturer_Name (none) -> Diodes Inc.; Manufacturer_Part_Number (none) -> AZ1117CH-3.3TRG1; Mouser Part Number (none) -> 621-AZ1117CH-3.3TRG1; Mouser Price/Stock (none) -> https://www.mouser.co.uk/ProductDetail/Diodes-Incorporated/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
- J2, J3: symbol Connector:Conn_01x03_Male -> Connector:Conn_01x03_Pin
- KF1, KF2: symbol MyLib:KF142V-5.0-4P -> Connector_Generic:Conn_01x04
- L1: symbol pspice:INDUCTOR -> MyLib:INDUCTOR
- U4: footprint DS9503P:TSO6C -> MyFootprints:TSO6C; symbol DS9503P:DS9503P -> MyLib:DS9503P; Availability In Stock -> Not in stock; Check_prices https://www.snapeda.com/parts/DS9503P+T&R/Analog+Devices/vi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 -> https://www.snapeda.com/parts/DS9503P+T/Analog+Devices/view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; MP DS9503P+T&amp;R -> DS9503P+T; Package None -> TSOC-6 Maxim; SnapEDA_Link https://www.snapeda.com/parts/DS9503P+T&R/Analog+Devices/vi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 -> https://www.snapeda.com/parts/DS9503P+T/Analog+Devices/view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
- renumbered D3 to D2, D4 to D3, Q4 to Q3, Q5 to Q4, R13 to R11, R14 to R12
Connections:
- net +5V: now also J5.1 (VBUS), R13.1
- net GND: now also D4.1 (K), J5.5 (GND), J5.S1 (SHIELD), J5.S2 (SHIELD), J5.S3 (SHIELD)
- net at U2.6 (UD-): now also J5.2 (D-)
- net at U2.5 (UD+): now also J5.3 (D+)
- net GPIO14: no longer names the net of U1.5 (GPIO14)
- new net: D4.2 (A), R13.2
- no-connect marks 12 -> 13
